Commit message: first commit

File: build/lib/gym_panda_reach/envs/base.urdf (robot description, URDF)
Before this commit: robot cube, 1 links, 0 joints
Links:
- link baseLink: geometry collision cylinder length=0.65 radius=0.2; visual cylinder length=0.65 radius=0.2

File: build/lib/gym_panda_reach/envs/floor.urdf (robot description, URDF)
Before this commit: robot cube, 1 links, 0 joints
Links:
- link baseLink: geometry collision box size=2 2 0.01; visual box size=2 2 0.01
